File: EAGLE Schematics and board files/Test Eagle File Sch.brd (EAGLE design)
At the start: 11 parts, among them IC1 LM317MBSTT3

Commit message: Things changed lol
Parts:
- added J1, J2, J3, J4, J5, J6, J7: 6_PIN_SERIAL_CABLEPTH, SparkFun-Connectors:FTDI_BASIC
Connections:
- new net V0: C1.1
Changed lines of the file:
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@@
 <attribute name="VALUE" x="-3.81" y="-57.15" size="1.27" layer="27"/>
+</element>
+<element name="J1" library="SparkFun-Connectors" library_urn="urn:adsk.eagle:library:513" package="FTDI_BASIC" value="6_PIN_SERIAL_CABLEPTH" x="-10.16" y="-63.5" smashed="yes">
+<attribute name="NAME" x="-5.588" y="-61.849" size="0.6096" layer="25" font="vector" ratio="20"/>
+<attribute name="VALUE" x="-5.588" y="-65.659" size="0.6096" layer="27" font="vector" ratio="20"/>
+</element>
+<element name="J2" library="SparkFun-Connectors" library_urn="urn:adsk.eagle:library:513" package="FTDI_BASIC" value="6_PIN_SERIAL_CABLEPTH" x="-10.16" y="-72.39" smashed="yes">
+<attribute name="NAME" x="-5.588" y="-70.739" size="0.6096" layer="25" font="vector" ratio="20"/>
+<attribute name="VALUE" x="-5.588" y="-74.549" size="0.6096" layer="27" font="vector" ratio="20"/>
+</element>
+<element name="J3" library="SparkFun-Connectors" library_urn="urn:adsk.eagle:library:513" package="FTDI_BASIC" value="6_PIN_SERIAL_CABLEPTH" x="-10.16" y="-81.28" smashed="yes">
+<attribute name="NAME" x="-5.588" y="-79.629" size="0.6096" layer="25" font="vector" ratio="20"/>
+<attribute name="VALUE" x="-5.588" y="-83.439" size="0.6096" layer="27" font="vector" ratio="20"/>
+</element>
+<element name="J4" library="SparkFun-Connectors" library_urn="urn:adsk.eagle:library:513" package="FTDI_BASIC" value="6_PIN_SERIAL_CABLEPTH" x="-10.16" y="-90.17" smashed="yes">
+<attribute name="NAME" x="-5.588" y="-88.519" size="0.6096" layer="25" font="vector" ratio="20"/>
+<attribute name="VALUE" x="-5.588" y="-92.329" size="0.6096" layer="27" font="vector" ratio="20"/>
+</element>
+<element name="J5" library="SparkFun-Connectors" library_urn="urn:adsk.eagle:library:513" package="FTDI_BASIC" value="6_PIN_SERIAL_CABLEPTH" x="-10.16" y="-99.06" smashed="yes">
+<attribute name="NAME" x="-5.588" y="-97.409" size="0.6096" layer="25" font="vector" ratio="20"/>
+<attribute name="VALUE" x="-5.588" y="-101.219" size="0.6096" layer="27" font="vector" ratio="20"/>
+</element>
+<element name="J6" library="SparkFun-Connectors" library_urn="urn:adsk.eagle:library:513" package="FTDI_BASIC" value="6_PIN_SERIAL_CABLEPTH" x="-10.16" y="-107.95" smashed="yes">
+<attribute name="NAME" x="-5.588" y="-106.299" size="0.6096" layer="25" font="vector" ratio="20"/>
+<attribute name="VALUE" x="-5.588" y="-110.109" size="0.6096" layer="27" font="vector" ratio="20"/>
+</element>
+<element name="J7" library="SparkFun-Connectors" library_urn="urn:adsk.eagle:library:513" package="FTDI_BASIC" value="6_PIN_SERIAL_CABLEPTH" x="-10.16" y="-116.84" smashed="yes">
+<attribute name="NAME" x="-5.588" y="-115.189" size="0.6096" layer="25" font="vector" ratio="20"/>
+<attribute name="VALUE" x="-5.588" y="-118.999" size="0.6096" layer="27" font="vector" ratio="20"/>
 </element>
 </elements>
@@
 <wire x1="5.08" y1="-39.37" x2="-5.32" y2="-41.25" width="0" layer="19" extent="1-1"/>
 </signal>
+<signal name="V0">
+<contactref element="C1" pad="1"/>
+</signal>
 </signals>
