File: EAGLE Schematics and board files/Test Eagle File Sch.brd (EAGLE design)
At the start: 11 parts, among them IC1 LM317MBSTT3

Commit message: Derp Derp :)
Derp Derp
Connections:
- new net N$3: C1.1
Changed lines of the file:
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@@
 <wire x1="5.08" y1="-39.37" x2="-5.32" y2="-41.25" width="0" layer="19" extent="1-1"/>
+</signal>
+<signal name="N$3">
+<contactref element="C1" pad="1"/>
 </signal>
 </signals>
