File: EAGLE Schematics and board files/Test Eagle File Sch.sch (EAGLE design)
At the start: 11 parts, among them IC1 LM317MBSTT3

Commit message: Things changed lol
Parts:
- added J1, J2, J3, J4, J5, J6, J7: 6_PIN_SERIAL_CABLEPTH, SparkFun-Connectors:6_PIN_SERIAL_CABLEPTH
Connections:
- new net V0: C1.1
Changed lines of the file:
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@@
 <part name="SUPPLY2" library="supply1" library_urn="urn:adsk.eagle:library:371" deviceset="GND" device=""/>
 <part name="SUPPLY4" library="supply1" library_urn="urn:adsk.eagle:library:371" deviceset="GND" device=""/>
+<part name="J1" library="SparkFun-Connectors" library_urn="urn:adsk.eagle:library:513" deviceset="6_PIN_SERIAL_CABLE" device="PTH"/>
+<part name="J2" library="SparkFun-Connectors" library_urn="urn:adsk.eagle:library:513" deviceset="6_PIN_SERIAL_CABLE" device="PTH"/>
+<part name="J3" library="SparkFun-Connectors" library_urn="urn:adsk.eagle:library:513" deviceset="6_PIN_SERIAL_CABLE" device="PTH"/>
+<part name="J4" library="SparkFun-Connectors" library_urn="urn:adsk.eagle:library:513" deviceset="6_PIN_SERIAL_CABLE" device="PTH"/>
+<part name="J5" library="SparkFun-Connectors" library_urn="urn:adsk.eagle:library:513" deviceset="6_PIN_SERIAL_CABLE" device="PTH"/>
+<part name="J6" library="SparkFun-Connectors" library_urn="urn:adsk.eagle:library:513" deviceset="6_PIN_SERIAL_CABLE" device="PTH"/>
+<part name="J7" library="SparkFun-Connectors" library_urn="urn:adsk.eagle:library:513" deviceset="6_PIN_SERIAL_CABLE" device="PTH"/>
 </parts>
 <sheets>
@@
 <wire x1="76.2" y1="58.42" x2="53.34" y2="58.42" width="0.1524" layer="91"/>
 <junction x="76.2" y="48.26"/>
+</segment>
+</net>
+<net name="V0" class="0">
+<segment>
+<pinref part="C1" gate="G$1" pin="1"/>
+<wire x1="53.34" y1="66.04" x2="53.34" y2="68.58" width="0.1524" layer="91"/>
+<wire x1="53.34" y1="68.58" x2="58.42" y2="68.58" width="0.1524" layer="91"/>
+<label x="55.88" y="68.58" size="1.778" layer="95"/>
 </segment>
 </net>
@@
 <attribute name="VALUE" x="109.22" y="22.86" size="1.778" layer="96"/>
 </instance>
+<instance part="J1" gate="G$1" x="30.48" y="20.32" smashed="yes">
+<attribute name="VALUE" x="25.4" y="10.414" size="1.778" layer="96" font="vector"/>
+<attribute name="NAME" x="25.4" y="30.988" size="1.778" layer="95" font="vector"/>
+</instance>
+<instance part="J2" gate="G$1" x="71.12" y="15.24" smashed="yes">
+<attribute name="VALUE" x="66.04" y="5.334" size="1.778" layer="96" font="vector"/>
+<attribute name="NAME" x="66.04" y="25.908" size="1.778" layer="95" font="vector"/>
+</instance>
+<instance part="J3" gate="G$1" x="104.14" y="12.7" smashed="yes">
+<attribute name="VALUE" x="99.06" y="2.794" size="1.778" layer="96" font="vector"/>
+<attribute name="NAME" x="99.06" y="23.368" size="1.778" layer="95" font="vector"/>
+</instance>
+<instance part="J4" gate="G$1" x="22.86" y="50.8" smashed="yes">
+<attribute name="VALUE" x="17.78" y="40.894" size="1.778" layer="96" font="vector"/>
+<attribute name="NAME" x="17.78" y="61.468" size="1.778" layer="95" font="vector"/>
+</instance>
+<instance part="J5" gate="G$1" x="40.64" y="45.72" smashed="yes">
+<attribute name="VALUE" x="35.56" y="35.814" size="1.778" layer="96" font="vector"/>
+<attribute name="NAME" x="35.56" y="56.388" size="1.778" layer="95" font="vector"/>
+</instance>
+<instance part="J6" gate="G$1" x="147.32" y="48.26" smashed="yes">
+<attribute name="VALUE" x="142.24" y="38.354" size="1.778" layer="96" font="vector"/>
+<attribute name="NAME" x="142.24" y="58.928" size="1.778" layer="95" font="vector"/>
+</instance>
+<instance part="J7" gate="G$1" x="182.88" y="43.18" smashed="yes">
+<attribute name="VALUE" x="177.8" y="33.274" size="1.778" layer="96" font="vector"/>
+<attribute name="NAME" x="177.8" y="53.848" size="1.778" layer="95" font="vector"/>
+</instance>
 </instances>
 <busses>
@@
 <segment>
 <pinref part="D2" gate="1" pin="C"/>
-<wire x1="96.52" y1="66.04" x2="96.52" y2="58.42" width="0.1524" layer="91"/>
-<wire x1="96.52" y1="66.04" x2="111.76" y2="66.04" width="0.1524" layer="91"/>
+<wire x1="93.98" y1="71.12" x2="96.52" y2="58.42" width="0.1524" layer="91"/>
+<wire x1="93.98" y1="71.12" x2="127" y2="71.12" width="0.1524" layer="91"/>
 <pinref part="IC1" gate="G$1" pin="OUT"/>
 <pinref part="R1" gate="G$1" pin="2"/>
-<wire x1="111.76" y1="66.04" x2="116.84" y2="66.04" width="0.1524" layer="91"/>
+<wire x1="127" y1="71.12" x2="134.62" y2="66.04" width="0.1524" layer="91"/>
 <wire x1="71.12" y1="66.04" x2="81.28" y2="66.04" width="0.1524" layer="91"/>
 <wire x1="81.28" y1="66.04" x2="81.28" y2="60.96" width="0.1524" layer="91"/>
-<wire x1="96.52" y1="66.04" x2="81.28" y2="66.04" width="0.1524" layer="91"/>
-<junction x="96.52" y="66.04"/>
+<wire x1="93.98" y1="71.12" x2="81.28" y2="66.04" width="0.1524" layer="91"/>
+<junction x="93.98" y="71.12"/>
 <junction x="81.28" y="66.04"/>
 <pinref part="D1" gate="1" pin="A"/>
@@
 <wire x1="81.28" y1="79.2" x2="81.28" y2="66.04" width="0.1524" layer="91"/>
 <pinref part="C5" gate="G$1" pin="+"/>
-<wire x1="111.76" y1="48.26" x2="111.76" y2="66.04" width="0.1524" layer="91"/>
-<junction x="111.76" y="66.04"/>
+<wire x1="111.76" y1="48.26" x2="127" y2="71.12" width="0.1524" layer="91"/>
+<junction x="127" y="71.12"/>
 <label x="116.84" y="68.58" size="1.778" layer="95"/>
-<junction x="116.84" y="66.04"/>
+<junction x="134.62" y="66.04"/>
+<label x="121.92" y="76.2" size="1.778" layer="95"/>
 </segment>
 </net>
@@
 <pinref part="C4" gate="G$1" pin="1"/>
 <pinref part="IC1" gate="G$1" pin="IN"/>
-<wire x1="55.88" y1="66.04" x2="53.34" y2="66.04" width="0.1524" layer="91"/>
-<wire x1="53.34" y1="66.04" x2="53.34" y2="48.26" width="0.1524" layer="91"/>
-<junction x="53.34" y="66.04"/>
-<wire x1="48.26" y1="66.04" x2="53.34" y2="66.04" width="0.1524" layer="91"/>
-<wire x1="53.34" y1="66.04" x2="53.34" y2="79.2" width="0.1524" layer="91"/>
+<wire x1="55.88" y1="66.04" x2="48.26" y2="66.04" width="0.1524" layer="91"/>
+<wire x1="48.26" y1="66.04" x2="53.34" y2="48.26" width="0.1524" layer="91"/>
+<junction x="48.26" y="66.04"/>
+<wire x1="43.18" y1="66.04" x2="48.26" y2="66.04" width="0.1524" layer="91"/>
+<wire x1="48.26" y1="66.04" x2="53.34" y2="79.2" width="0.1524" layer="91"/>
 <pinref part="D1" gate="1" pin="C"/>
 <wire x1="60.96" y1="79.2" x2="53.34" y2="79.2" width="0.1524" layer="91"/>
 <label x="48.26" y="68.58" size="1.778" layer="95" rot="MR0"/>
-<junction x="48.26" y="66.04"/>
-</segment>
-</net>
+<junction x="43.18" y="66.04"/>
+</segment>
+</net>
